Commit message: urdf: fine-tune for our fingers
Signed-off-by: Wolfgang Wiedmeyer <wolfgang.wiedmeyer@kit.edu>

File: urdf/egl90_macro.xacro (robot description, xacro)
@@ -13,5 +13,5 @@
       <parent link="${prefix}jaw_base"/>
       <child link="${prefix}finger_right"/>
-      <origin rpy="0.0 0.0 ${pi}" xyz="${x} -0.0255 -0.018"/>
+      <origin rpy="0.0 0.0 ${pi}" xyz="${x - 0.065} -0.013 -0.018"/>
       <axis xyz="1 0 0"/>
       <limit effort="100.0" lower="${min}" upper="${max}" velocity="100.0"/>
@@ -19,12 +19,14 @@
     <link name="${prefix}finger_right">
       <visual>
+        <origin xyz="0 0 0" rpy="${90 * PI / 180} 0 ${90 * PI / 180}"/>
         <geometry>
           <xacro:insert_block name="mesh"/>
         </geometry>
-        <material name="grey ">
-          <color rgba="0.5 0.5 0.5 1.0"/>
+        <material name="black ">
+          <color rgba="1.0 1.0 1.0 1.0"/>
         </material>
       </visual>
       <collision>
+        <origin xyz="0 0 0" rpy="${90 * PI / 180} 0 ${90 * PI / 180}"/>
         <geometry>
           <xacro:insert_block name="mesh"/>
@@ -35,5 +37,5 @@
       <parent link="${prefix}jaw_base"/>
       <child link="${prefix}finger_left"/>
-      <origin rpy="0.0 0.0 0.0" xyz="${x} 0.0255 -0.018"/>
+      <origin rpy="0.0 0.0 0.0" xyz="${x + 0.065} 0.013 -0.018"/>
       <axis xyz="1 0 0"/>
       <limit effort="100.0" lower="${min}" upper="${max}" velocity="100.0"/>
@@ -42,12 +44,14 @@
     <link name="${prefix}finger_left">
       <visual>
+        <origin xyz="0 0 0" rpy="${90 * PI / 180} 0 ${90 * PI / 180}"/>
         <geometry>
           <xacro:insert_block name="mesh"/>
         </geometry>
-        <material name="grey ">
-          <color rgba="0.5 0.5 0.5 1.0"/>
+        <material name="black ">
+          <color rgba="1.0 1.0 1.0 1.0"/>
         </material>
       </visual>
       <collision>
+        <origin xyz="0 0 0" rpy="${90 * PI / 180} 0 ${90 * PI / 180}"/>
         <geometry>
           <xacro:insert_block name="mesh"/>

Commit message: HACK: set gripper joints fixed at open position
Signed-off-by: Wolfgang Wiedmeyer <wolfgang.wiedmeyer@kit.edu>

File: urdf/egl90_macro.xacro (robot description, xacro)
@@ -10,8 +10,8 @@
   <xacro:property name="jaw_base_z" value="0.0191"/>
   <xacro:macro name="egl90-jaws" params="prefix x min max *mesh">
-    <joint name="egl_position" type="prismatic">
+    <joint name="egl_position" type="fixed">
       <parent link="${prefix}jaw_base"/>
       <child link="${prefix}finger_right"/>
-      <origin rpy="0.0 0.0 ${pi}" xyz="${x - 0.065} -0.013 -0.018"/>
+      <origin rpy="0.0 0.0 ${pi}" xyz="${x - 0.1} -0.013 -0.018"/>
       <axis xyz="1 0 0"/>
       <limit effort="100.0" lower="${min}" upper="${max}" velocity="100.0"/>
@@ -34,8 +34,8 @@
       </collision>
     </link>
-    <joint name="egl_position_mimic" type="prismatic">
+    <joint name="egl_position_mimic" type="fixed">
       <parent link="${prefix}jaw_base"/>
       <child link="${prefix}finger_left"/>
-      <origin rpy="0.0 0.0 0.0" xyz="${x + 0.065} 0.013 -0.018"/>
+      <origin rpy="0.0 0.0 0.0" xyz="${x + 0.1} 0.013 -0.018"/>
       <axis xyz="1 0 0"/>
       <limit effort="100.0" lower="${min}" upper="${max}" velocity="100.0"/>

Commit message: urdf: fine-tune finger position
Signed-off-by: Wolfgang Wiedmeyer <wolfgang.wiedmeyer@kit.edu>

File: urdf/egl90_macro.xacro (robot description, xacro)
@@ -13,5 +13,5 @@
       <parent link="${prefix}jaw_base"/>
       <child link="${prefix}finger_right"/>
-      <origin rpy="0.0 0.0 ${pi}" xyz="${x - 0.1} -0.013 -0.018"/>
+      <origin rpy="0.0 0.0 ${pi}" xyz="${x - 0.1} -0.013 0.005"/>
       <axis xyz="1 0 0"/>
       <limit effort="100.0" lower="${min}" upper="${max}" velocity="100.0"/>
@@ -37,5 +37,5 @@
       <parent link="${prefix}jaw_base"/>
       <child link="${prefix}finger_left"/>
-      <origin rpy="0.0 0.0 0.0" xyz="${x + 0.1} 0.013 -0.018"/>
+      <origin rpy="0.0 0.0 0.0" xyz="${x + 0.1} 0.013 0.005"/>
       <axis xyz="1 0 0"/>
       <limit effort="100.0" lower="${min}" upper="${max}" velocity="100.0"/>
